Commit message: cambios a urdf, tenemos automatizados los experimentos, graficos de corridas y plotter

File: URDF/nashe.urdf (robot description, URDF)
Before this commit: robot youBot, 10 links, 9 joints
Links:
- removed link base_link_gt
- added link base_link, mass 10.0; collision box size=0.006898 0.026477 0.075109; collision box size=0.006898 0.026477 0.075109
Joints:
- joint Joint: parent base_link_gt -> base_link
- joint rollingJoint_rl: parent base_link_gt -> base_link
- joint rollingJoint_rr: parent base_link_gt -> base_link
